File: master.sch (EAGLE design)
At the start: 9 parts

Commit message: poprawione polaczenia, usunieta masa pod antena,
Parts:
- removed JP2: (no value), pinhead:PINHD-1X3/90
- added R3: 47k, rcl:R-EU_M0805
- added R4: 100k, rcl:R-EU_M0805
Connections:
- removed net RX: JP2.2, U$2.RX
- removed net TX: JP2.3, U$2.TX
- new net RST: R4.2, U$2.RST
- net +3V3: now also R4.1, S1.NO
- net BUTTON: now also R3.1, U$2.D8; no longer U$2.D0
- net GND: now also R3.2; no longer JP2.1, S1.NO
- net INTERRUPT: now also U$2.D0; no longer U$2.D8
Other:
- note removed: "UART"
- moved on the sheet: S1
Changed lines of the file:
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@@
 <layer number="91" name="Nets" color="2" fill="1" visible="yes" active="yes"/>
 <layer number="92" name="Busses" color="1" fill="1" visible="yes" active="yes"/>
-<layer number="93" name="Pins" color="2" fill="1" visible="yes" active="yes"/>
+<layer number="93" name="Pins" color="2" fill="1" visible="no" active="yes"/>
 <layer number="94" name="Symbols" color="4" fill="1" visible="yes" active="yes"/>
 <layer number="95" name="Names" color="7" fill="1" visible="yes" active="yes"/>
@@
 <clearance class="0" value="0.127"/>
 </class>
-<class number="1" name="vcc" width="0.508" drill="0">
-<clearance class="1" value="0.1524"/>
+<class number="1" name="vcc" width="0.5" drill="0">
+<clearance class="1" value="0.127"/>
 </class>
 </classes>
@@
 <part name="GND1" library="supply1" library_urn="urn:adsk.eagle:library:371" deviceset="GND" device=""/>
 <part name="GND7" library="supply1" library_urn="urn:adsk.eagle:library:371" deviceset="GND" device=""/>
-<part name="JP2" library="pinhead" library_urn="urn:adsk.eagle:library:325" deviceset="PINHD-1X3" device="/90" package3d_urn="urn:adsk.eagle:package:22459/2"/>
 <part name="R2" library="rcl" library_urn="urn:adsk.eagle:library:334" deviceset="R-EU_" device="M0805" package3d_urn="urn:adsk.eagle:package:23556/2" value="10Ohm"/>
 <part name="S1" library="Modules" deviceset="TS-1187A-B-A-B" device="" package3d_urn="urn:adsk.eagle:package:24754950/2"/>
-<part name="GND2" library="supply1" library_urn="urn:adsk.eagle:library:371" deviceset="GND" device=""/>
+<part name="R3" library="rcl" library_urn="urn:adsk.eagle:library:334" deviceset="R-EU_" device="M0805" package3d_urn="urn:adsk.eagle:package:23556/2" value="47k"/>
+<part name="+3V2" library="supply1" library_urn="urn:adsk.eagle:library:371" deviceset="+3V3" device=""/>
+<part name="+3V3" library="supply1" library_urn="urn:adsk.eagle:library:371" deviceset="+3V3" device=""/>
+<part name="R4" library="rcl" library_urn="urn:adsk.eagle:library:334" deviceset="R-EU_" device="M0805" package3d_urn="urn:adsk.eagle:package:23556/2" value="100k"/>
 </parts>
 <sheets>
@@
 <wire x1="73.66" y1="-15.24" x2="96.52" y2="-15.24" width="0.254" layer="97"/>
 <text x="76.2" y="50.8" size="2.54" layer="97">LED 1</text>
-<text x="22.86" y="-20.32" size="2.54" layer="97">UART</text>
-<wire x1="20.32" y1="-15.24" x2="20.32" y2="-38.1" width="0.254" layer="97"/>
-<wire x1="20.32" y1="-38.1" x2="96.52" y2="-38.1" width="0.254" layer="97"/>
-<wire x1="96.52" y1="-38.1" x2="96.52" y2="-15.24" width="0.254" layer="97"/>
 <wire x1="-119.38" y1="5.08" x2="-119.38" y2="-48.26" width="0.254" layer="97"/>
 <wire x1="-119.38" y1="-48.26" x2="-17.78" y2="-48.26" width="0.254" layer="97"/>
@@
 <attribute name="VALUE" x="-76.2" y="-7.62" size="1.778" layer="96"/>
 </instance>
-<instance part="+3V4" gate="G$1" x="-106.68" y="-30.48" smashed="yes">
-<attribute name="VALUE" x="-104.14" y="-30.48" size="1.778" layer="96"/>
+<instance part="+3V4" gate="G$1" x="-114.3" y="-30.48" smashed="yes">
+<attribute name="VALUE" x="-111.76" y="-30.48" size="1.778" layer="96"/>
 </instance>
 <instance part="GND1" gate="1" x="-30.48" y="-33.02" smashed="yes">
 <attribute name="VALUE" x="-33.02" y="-35.56" size="1.778" layer="96"/>
 </instance>
-<instance part="GND7" gate="1" x="60.96" y="-7.62" smashed="yes">
-<attribute name="VALUE" x="58.42" y="-10.16" size="1.778" layer="96"/>
-</instance>
-<instance part="JP2" gate="A" x="71.12" y="-27.94" smashed="yes">
-<attribute name="NAME" x="64.77" y="-22.225" size="1.778" layer="95"/>
-<attribute name="VALUE" x="64.77" y="-35.56" size="1.778" layer="96"/>
+<instance part="GND7" gate="1" x="48.26" y="7.62" smashed="yes">
+<attribute name="VALUE" x="45.72" y="5.08" size="1.778" layer="96"/>
 </instance>
 <instance part="R2" gate="G$1" x="83.82" y="7.62" smashed="yes" rot="R90">
@@
 <attribute name="VALUE" x="87.122" y="3.81" size="1.778" layer="96" rot="R90"/>
 </instance>
-<instance part="S1" gate="G$1" x="50.8" y="2.54" smashed="yes">
-<attribute name="NAME" x="48.26" y="5.08" size="1.27" layer="95"/>
-</instance>
-<instance part="GND2" gate="1" x="43.18" y="-27.94" smashed="yes">
-<attribute name="VALUE" x="40.64" y="-30.48" size="1.778" layer="96"/>
+<instance part="S1" gate="G$1" x="53.34" y="-2.54" smashed="yes">
+<attribute name="NAME" x="50.8" y="0" size="1.27" layer="95"/>
+</instance>
+<instance part="R3" gate="G$1" x="40.64" y="5.08" smashed="yes" rot="R90">
+<attribute name="NAME" x="39.1414" y="3.81" size="1.778" layer="95" rot="R90"/>
+<attribute name="VALUE" x="43.942" y="3.81" size="1.778" layer="96" rot="R90"/>
+</instance>
+<instance part="+3V2" gate="G$1" x="68.58" y="5.08" smashed="yes">
+<attribute name="VALUE" x="66.04" y="0" size="1.778" layer="96" rot="R90"/>
+</instance>
+<instance part="+3V3" gate="G$1" x="-99.06" y="-7.62" smashed="yes">
+<attribute name="VALUE" x="-96.52" y="-7.62" size="1.778" layer="96"/>
+</instance>
+<instance part="R4" gate="G$1" x="-91.44" y="-15.24" smashed="yes">
+<attribute name="NAME" x="-95.25" y="-13.7414" size="1.778" layer="95"/>
+<attribute name="VALUE" x="-90.17" y="-13.462" size="1.778" layer="96"/>
 </instance>
 </instances>
@@
 <segment>
 <pinref part="U$2" gate="G$1" pin="3V3"/>
-<wire x1="-81.28" y1="-33.02" x2="-106.68" y2="-33.02" width="0.1524" layer="91"/>
+<wire x1="-81.28" y1="-33.02" x2="-114.3" y2="-33.02" width="0.1524" layer="91"/>
 <pinref part="+3V4" gate="G$1" pin="+3V3"/>
+</segment>
+<segment>
+<pinref part="R4" gate="G$1" pin="1"/>
+<pinref part="+3V3" gate="G$1" pin="+3V3"/>
+<wire x1="-96.52" y1="-15.24" x2="-99.06" y2="-15.24" width="0.1524" layer="91"/>
+<wire x1="-99.06" y1="-15.24" x2="-99.06" y2="-10.16" width="0.1524" layer="91"/>
+</segment>
+<segment>
+<pinref part="S1" gate="G$1" pin="NO"/>
+<pinref part="+3V2" gate="G$1" pin="+3V3"/>
+<wire x1="60.96" y1="-2.54" x2="68.58" y2="-2.54" width="0.1524" layer="91"/>
+<wire x1="68.58" y1="-2.54" x2="68.58" y2="2.54" width="0.1524" layer="91"/>
 </segment>
 </net>
@@
 <segment>
 <pinref part="GND7" gate="1" pin="GND"/>
-<pinref part="S1" gate="G$1" pin="NO"/>
-<wire x1="58.42" y1="2.54" x2="60.96" y2="2.54" width="0.1524" layer="91"/>
-<wire x1="60.96" y1="2.54" x2="60.96" y2="-5.08" width="0.1524" layer="91"/>
-</segment>
-<segment>
-<pinref part="JP2" gate="A" pin="1"/>
-<wire x1="68.58" y1="-25.4" x2="43.18" y2="-25.4" width="0.1524" layer="91"/>
-<pinref part="GND2" gate="1" pin="GND"/>
+<wire x1="48.26" y1="10.16" x2="48.26" y2="12.7" width="0.1524" layer="91"/>
+<pinref part="R3" gate="G$1" pin="2"/>
+<wire x1="48.26" y1="12.7" x2="40.64" y2="12.7" width="0.1524" layer="91"/>
+<wire x1="40.64" y1="12.7" x2="40.64" y2="10.16" width="0.1524" layer="91"/>
 </segment>
 </net>
@@
 <net name="BUTTON" class="0">
 <segment>
-<wire x1="22.86" y1="2.54" x2="43.18" y2="2.54" width="0.1524" layer="91"/>
-<label x="22.86" y="2.54" size="1.778" layer="95"/>
+<wire x1="22.86" y1="-2.54" x2="40.64" y2="-2.54" width="0.1524" layer="91"/>
+<label x="22.86" y="-2.54" size="1.778" layer="95"/>
 <pinref part="S1" gate="G$1" pin="COM"/>
+<wire x1="40.64" y1="-2.54" x2="45.72" y2="-2.54" width="0.1524" layer="91"/>
+<pinref part="R3" gate="G$1" pin="1"/>
+<wire x1="40.64" y1="0" x2="40.64" y2="-2.54" width="0.1524" layer="91"/>
+<junction x="40.64" y="-2.54"/>
+</segment>
+<segment>
+<pinref part="U$2" gate="G$1" pin="D8"/>
+<wire x1="-81.28" y1="-30.48" x2="-99.06" y2="-30.48" width="0.1524" layer="91"/>
+<label x="-99.06" y="-30.48" size="1.778" layer="95"/>
+</segment>
+</net>
+<net name="INTERRUPT" class="0">
+<segment>
+<pinref part="NRF24" gate="G$1" pin="8.IRQ"/>
+<wire x1="-88.9" y1="12.7" x2="-45.72" y2="12.7" width="0.1524" layer="91"/>
+<label x="-88.9" y="12.7" size="1.778" layer="95" rot="R180" xref="yes"/>
 </segment>
 <segment>
@@
 <wire x1="-81.28" y1="-20.32" x2="-99.06" y2="-20.32" width="0.1524" layer="91"/>
 <label x="-99.06" y="-20.32" size="1.778" layer="95"/>
-</segment>
-</net>
-<net name="INTERRUPT" class="0">
-<segment>
-<pinref part="U$2" gate="G$1" pin="D8"/>
-<wire x1="-81.28" y1="-30.48" x2="-99.06" y2="-30.48" width="0.1524" layer="91"/>
-<label x="-99.06" y="-30.48" size="1.778" layer="95"/>
-</segment>
-<segment>
-<pinref part="NRF24" gate="G$1" pin="8.IRQ"/>
-<wire x1="-88.9" y1="12.7" x2="-45.72" y2="12.7" width="0.1524" layer="91"/>
-<label x="-88.9" y="12.7" size="1.778" layer="95" rot="R180" xref="yes"/>
 </segment>
 </net>
@@
 </segment>
 </net>
-<net name="TX" class="0">
-<segment>
-<pinref part="U$2" gate="G$1" pin="TX"/>
-<wire x1="-30.48" y1="-15.24" x2="-45.72" y2="-15.24" width="0.1524" layer="91"/>
-<label x="-38.1" y="-15.24" size="1.778" layer="95"/>
-</segment>
-<segment>
-<pinref part="JP2" gate="A" pin="3"/>
-<wire x1="68.58" y1="-30.48" x2="50.8" y2="-30.48" width="0.1524" layer="91"/>
-<label x="50.8" y="-30.48" size="1.778" layer="95"/>
-</segment>
-</net>
-<net name="RX" class="0">
-<segment>
-<pinref part="U$2" gate="G$1" pin="RX"/>
-<wire x1="-45.72" y1="-17.78" x2="-30.48" y2="-17.78" width="0.1524" layer="91"/>
-<label x="-38.1" y="-17.78" size="1.778" layer="95"/>
-</segment>
-<segment>
-<pinref part="JP2" gate="A" pin="2"/>
-<wire x1="68.58" y1="-27.94" x2="50.8" y2="-27.94" width="0.1524" layer="91"/>
-<label x="50.8" y="-27.94" size="1.778" layer="95"/>
-</segment>
-</net>
 <net name="N$3" class="0">
 <segment>
@@
 </segment>
 </net>
+<net name="RST" class="0">
+<segment>
+<pinref part="U$2" gate="G$1" pin="RST"/>
+<pinref part="R4" gate="G$1" pin="2"/>
+<wire x1="-81.28" y1="-15.24" x2="-86.36" y2="-15.24" width="0.1524" layer="91"/>
+<label x="-81.28" y="-15.24" size="1.778" layer="95"/>
+</segment>
+</net>
